Commit message: add camera

File: assembler/techtory_cobotta_description/urdf/techtory_cobotta.urdf.xacro (robot description, xacro)
@@ -23,20 +23,56 @@
         <origin xyz="0 0 0" rpy="0 0 0" />
     </joint>
-    <!-- Dummy Camera -->
-    <link name="$(arg prefix)camera_link">
-        <visual>
-            <geometry>
-                <box size="0.05 0.05 0.05" />
-            </geometry>
-            <material name="black">
-                <color rgba="0 0 0 1" />
-            </material>
-        </visual>
-    </link>
-    <joint name="$(arg prefix)camera_joint" type="fixed">
-        <parent link="$(arg prefix)cell_link" />
-        <child link="$(arg prefix)camera_link" />
-        <origin xyz="0.5 0 1.5" rpy="0 ${pi/2} 0" />
-    </joint>
+    <!-- RealSense Cameras -->
+    <xacro:include filename="$(find realsense2_description)/urdf/_d435.urdf.xacro"/>
+    <xacro:sensor_d435 parent="$(arg prefix)cell_link" name="$(arg prefix)camera1" use_nominal_extrinsics="true">
+        <origin xyz="0.65 0.65 2.0" rpy="0 ${3*pi/4} ${pi/4}" />
+    </xacro:sensor_d435>
+    <xacro:sensor_d435 parent="$(arg prefix)cell_link" name="$(arg prefix)camera2" use_nominal_extrinsics="true">
+        <origin xyz="-0.65 0.65 2.0" rpy="0 ${pi/4} -${pi/4}" />
+    </xacro:sensor_d435>
+    <xacro:if value="${'$(arg sim_type)' == 'gazebo'}">
+        <gazebo reference="$(arg prefix)camera1_link">
+            <sensor name="$(arg prefix)camera1" type="rgbd_camera">
+                <camera>
+                    <horizontal_fov>1.204</horizontal_fov>
+                    <image>
+                        <width>640</width>
+                        <height>480</height>
+                        <format>R8G8B8</format>
+                    </image>
+                    <clip>
+                        <near>0.1</near>
+                        <far>10.0</far>
+                    </clip>
+                </camera>
+                <always_on>1</always_on>
+                <update_rate>30</update_rate>
+                <visualize>true</visualize>
+                <topic>$(arg prefix)camera1</topic>
+                <gz_frame_id>$(arg prefix)camera1_link</gz_frame_id>
+            </sensor>
+        </gazebo>
+        <gazebo reference="$(arg prefix)camera2_link">
+            <sensor name="$(arg prefix)camera2" type="rgbd_camera">
+                <camera>
+                    <horizontal_fov>1.204</horizontal_fov>
+                    <image>
+                        <width>640</width>
+                        <height>480</height>
+                        <format>R8G8B8</format>
+                    </image>
+                    <clip>
+                        <near>0.1</near>
+                        <far>10.0</far>
+                    </clip>
+                </camera>
+                <always_on>1</always_on>
+                <update_rate>30</update_rate>
+                <visualize>true</visualize>
+                <topic>$(arg prefix)camera2</topic>
+                <gz_frame_id>$(arg prefix)camera2_link</gz_frame_id>
+            </sensor>
+        </gazebo>
+    </xacro:if>
     <!-- ROS 2 Control Instance -->
     <xacro:techtory_cobotta_ros2_control

File: assembler/techtory_franka_description/urdf/techtory_franka.urdf (robot description, URDF)
Before this commit: robot techtory_franka, 29 links, 28 joints
Links:
- removed link camera_link
- added link camera1_bottom_screw_frame
- added link camera1_link
- added link camera2_bottom_screw_frame
- added link camera2_link
Joints:
- removed joint camera_joint
- added joint camera1_joint: type fixed, parent cell_link, child camera1_bottom_screw_frame, origin xyz=0.65 0.65 2.0 rpy=0 2.356194490192345 0.7853981633974483
- added joint camera1_link_joint: type fixed, parent camera1_bottom_screw_frame, child camera1_link, origin xyz=0.010600000000000002 0.0175 0.0125 rpy=0 0 0
- added joint camera2_joint: type fixed, parent cell_link, child camera2_bottom_screw_frame, origin xyz=-0.65 0.65 2.0 rpy=0 0.7853981633974483 -0.7853981633974483
- added joint camera2_link_joint: type fixed, parent camera2_bottom_screw_frame, child camera2_link, origin xyz=0.010600000000000002 0.0175 0.0125 rpy=0 0 0

File: assembler/techtory_franka_description/urdf/techtory_franka.urdf.xacro (robot description, xacro)
@@ -38,4 +38,56 @@
         <origin xyz="0 0 0" rpy="0 0 1.5708" />
     </joint>
+    <!-- RealSense Cameras -->
+    <xacro:include filename="$(find realsense2_description)/urdf/_d435.urdf.xacro"/>
+    <xacro:sensor_d435 parent="$(arg prefix)cell_link" name="$(arg prefix)camera1" use_nominal_extrinsics="true">
+        <origin xyz="0.65 0.65 2.0" rpy="0 ${3*pi/4} ${pi/4}" />
+    </xacro:sensor_d435>
+    <xacro:sensor_d435 parent="$(arg prefix)cell_link" name="$(arg prefix)camera2" use_nominal_extrinsics="true">
+        <origin xyz="-0.65 0.65 2.0" rpy="0 ${pi/4} -${pi/4}" />
+    </xacro:sensor_d435>
+    <xacro:if value="${'$(arg sim_type)' == 'gazebo'}">
+        <gazebo reference="$(arg prefix)camera1_link">
+            <sensor name="$(arg prefix)camera1" type="rgbd_camera">
+                <camera>
+                    <horizontal_fov>1.204</horizontal_fov>
+                    <image>
+                        <width>640</width>
+                        <height>480</height>
+                        <format>R8G8B8</format>
+                    </image>
+                    <clip>
+                        <near>0.1</near>
+                        <far>10.0</far>
+                    </clip>
+                </camera>
+                <always_on>1</always_on>
+                <update_rate>30</update_rate>
+                <visualize>true</visualize>
+                <topic>$(arg prefix)camera1</topic>
+                <gz_frame_id>$(arg prefix)camera1_link</gz_frame_id>
+            </sensor>
+        </gazebo>
+        <gazebo reference="$(arg prefix)camera2_link">
+            <sensor name="$(arg prefix)camera2" type="rgbd_camera">
+                <camera>
+                    <horizontal_fov>1.204</horizontal_fov>
+                    <image>
+                        <width>640</width>
+                        <height>480</height>
+                        <format>R8G8B8</format>
+                    </image>
+                    <clip>
+                        <near>0.1</near>
+                        <far>10.0</far>
+                    </clip>
+                </camera>
+                <always_on>1</always_on>
+                <update_rate>30</update_rate>
+                <visualize>true</visualize>
+                <topic>$(arg prefix)camera2</topic>
+                <gz_frame_id>$(arg prefix)camera2_link</gz_frame_id>
+            </sensor>
+        </gazebo>
+    </xacro:if>
     <!-- ROS 2 Control Instance -->
     <xacro:techtory_franka_ros2_control
@@ -44,19 +96,3 @@
         robot_type="$(arg robot_type)"
         sim_type="$(arg sim_type)" />
-    <!-- Dummy Camera -->
-    <link name="$(arg prefix)camera_link">
-        <visual>
-            <geometry>
-                <box size="0.05 0.05 0.05" />
-            </geometry>
-            <material name="black">
-                <color rgba="0 0 0 1" />
-            </material>
-        </visual>
-    </link>
-    <joint name="$(arg prefix)camera_joint" type="fixed">
-        <parent link="$(arg prefix)cell_link" />
-        <child link="$(arg prefix)camera_link" />
-        <origin xyz="0.5 0 1.5" rpy="0 ${pi/2} 0" />
-    </joint>
 </robot>

File: assembler/techtory_ur5e_description/urdf/techtory_ur5e.urdf.xacro (robot description, xacro)
@@ -31,20 +31,56 @@
         <origin xyz="0 0 0" rpy="0 0 0" />
     </xacro:ur_robot>
-    <!-- Dummy Camera -->
-    <link name="$(arg prefix)camera_link">
-        <visual>
-            <geometry>
-                <box size="0.05 0.05 0.05" />
-            </geometry>
-            <material name="black">
-                <color rgba="0 0 0 1" />
-            </material>
-        </visual>
-    </link>
-    <joint name="$(arg prefix)camera_joint" type="fixed">
-        <parent link="$(arg prefix)cell_link" />
-        <child link="$(arg prefix)camera_link" />
-        <origin xyz="0.5 0 1.5" rpy="0 ${pi/2} 0" />
-    </joint>
+    <!-- RealSense Cameras -->
+    <xacro:include filename="$(find realsense2_description)/urdf/_d435.urdf.xacro"/>
+    <xacro:sensor_d435 parent="$(arg prefix)cell_link" name="$(arg prefix)camera1" use_nominal_extrinsics="true">
+        <origin xyz="0.65 0.65 2.0" rpy="0 ${3*pi/4} ${pi/4}" />
+    </xacro:sensor_d435>
+    <xacro:sensor_d435 parent="$(arg prefix)cell_link" name="$(arg prefix)camera2" use_nominal_extrinsics="true">
+        <origin xyz="-0.65 0.65 2.0" rpy="0 ${pi/4} -${pi/4}" />
+    </xacro:sensor_d435>
+    <xacro:if value="${'$(arg sim_type)' == 'gazebo'}">
+        <gazebo reference="$(arg prefix)camera1_link">
+            <sensor name="$(arg prefix)camera1" type="rgbd_camera">
+                <camera>
+                    <horizontal_fov>1.204</horizontal_fov>
+                    <image>
+                        <width>640</width>
+                        <height>480</height>
+                        <format>R8G8B8</format>
+                    </image>
+                    <clip>
+                        <near>0.1</near>
+                        <far>10.0</far>
+                    </clip>
+                </camera>
+                <always_on>1</always_on>
+                <update_rate>30</update_rate>
+                <visualize>true</visualize>
+                <topic>$(arg prefix)camera1</topic>
+                <gz_frame_id>$(arg prefix)camera1_link</gz_frame_id>
+            </sensor>
+        </gazebo>
+        <gazebo reference="$(arg prefix)camera2_link">
+            <sensor name="$(arg prefix)camera2" type="rgbd_camera">
+                <camera>
+                    <horizontal_fov>1.204</horizontal_fov>
+                    <image>
+                        <width>640</width>
+                        <height>480</height>
+                        <format>R8G8B8</format>
+                    </image>
+                    <clip>
+                        <near>0.1</near>
+                        <far>10.0</far>
+                    </clip>
+                </camera>
+                <always_on>1</always_on>
+                <update_rate>30</update_rate>
+                <visualize>true</visualize>
+                <topic>$(arg prefix)camera2</topic>
+                <gz_frame_id>$(arg prefix)camera2_link</gz_frame_id>
+            </sensor>
+        </gazebo>
+    </xacro:if>
     <!-- ROS 2 Control Instance -->
     <xacro:techtory_ur5e_ros2_control
