Commit message: Remove obsolete USD files and update initial positions for the Techtory Franka robot configuration
- Deleted unnecessary USD files related to materials, robot description, and the main USD file for the Techtory Franka robot.
- Updated initial joint positions in the MoveIt configuration to reflect more accurate values for fr3_joint1, fr3_joint2, fr3_joint4, fr3_joint6, and fr3_joint7.

File: assembler/techtory_franka_description/urdf/techtory_franka.ros2_control.xacro (robot description, xacro)
@@ -77,6 +77,10 @@
                 <state_interface name="velocity"/>
             </joint>
-            <!-- finger_joint2 mimics finger_joint1 — mimic joints must not have command interfaces -->
+            <!-- finger_joint2 mimics finger_joint1 — no command interface (enforced by ros2_control).
+                 The <param name="mimic"> tells topic_based_ros2_control to compute and publish its
+                 command value so Isaac Sim receives equal-length arrays for all 9 actuators. -->
             <joint name="${prefix}${robot_type}_finger_joint2">
+                <param name="mimic">${prefix}${robot_type}_finger_joint1</param>
+                <param name="multiplier">1</param>
                 <state_interface name="position">
                   <param name="initial_value">0.0</param>

File: assembler/techtory_franka_description/urdf/techtory_franka.urdf.xacro (robot description, xacro)
@@ -39,55 +39,16 @@
     </joint>
     <!-- RealSense Cameras -->
-    <xacro:include filename="$(find realsense2_description)/urdf/_d435.urdf.xacro"/>
-    <xacro:sensor_d435 parent="$(arg prefix)cell_link" name="$(arg prefix)camera1" use_nominal_extrinsics="true">
-        <origin xyz="0.65 0.65 2.0" rpy="0 ${3*pi/4} ${pi/4}" />
-    </xacro:sensor_d435>
-    <xacro:sensor_d435 parent="$(arg prefix)cell_link" name="$(arg prefix)camera2" use_nominal_extrinsics="true">
-        <origin xyz="-0.65 0.65 2.0" rpy="0 ${pi/4} -${pi/4}" />
-    </xacro:sensor_d435>
-    <xacro:if value="${'$(arg sim_type)' == 'gazebo'}">
-        <gazebo reference="$(arg prefix)camera1_link">
-            <sensor name="$(arg prefix)camera1" type="rgbd_camera">
-                <camera>
-                    <horizontal_fov>1.204</horizontal_fov>
-                    <image>
-                        <width>640</width>
-                        <height>480</height>
-                        <format>R8G8B8</format>
-                    </image>
-                    <clip>
-                        <near>0.1</near>
-                        <far>10.0</far>
-                    </clip>
-                </camera>
-                <always_on>1</always_on>
-                <update_rate>30</update_rate>
-                <visualize>true</visualize>
-                <topic>$(arg prefix)camera1</topic>
-                <gz_frame_id>$(arg prefix)camera1_link</gz_frame_id>
-            </sensor>
-        </gazebo>
-        <gazebo reference="$(arg prefix)camera2_link">
-            <sensor name="$(arg prefix)camera2" type="rgbd_camera">
-                <camera>
-                    <horizontal_fov>1.204</horizontal_fov>
-                    <image>
-                        <width>640</width>
-                        <height>480</height>
-                        <format>R8G8B8</format>
-                    </image>
-                    <clip>
-                        <near>0.1</near>
-                        <far>10.0</far>
-                    </clip>
-                </camera>
-                <always_on>1</always_on>
-                <update_rate>30</update_rate>
-                <visualize>true</visualize>
-                <topic>$(arg prefix)camera2</topic>
-                <gz_frame_id>$(arg prefix)camera2_link</gz_frame_id>
-            </sensor>
-        </gazebo>
-    </xacro:if>
+    <joint name="camera1_joint" type="fixed">
+        <origin rpy="0 2.356194490192345 0.7853981633974483" xyz="0.65 0.65 2.0"/>
+        <parent link="cell_link"/>
+        <child link="camera1_frame"/>
+    </joint>
+    <link name="camera1_frame"/>
+    <joint name="camera2_joint" type="fixed">
+        <origin rpy="0 0.7853981633974483 -0.7853981633974483" xyz="-0.65 0.65 2.0"/>
+        <parent link="cell_link"/>
+        <child link="camera2_frame"/>
+    </joint>
+    <link name="camera2_frame"/>
     <!-- ROS 2 Control Instance -->
     <xacro:techtory_franka_ros2_control
