Commit message: Add shelf and techtory demo description assets
- Created URDF and USD files for a shelf object, including its configuration and physics properties.
- Added techtory demo description URDF and corresponding USD configuration files.
- Implemented launch file for assembling the techtory workcell with the FR3 robot and shelf.
- Developed Python scripts for scene assembly in Isaac Sim, including spawners for the workcell and robot.
- Updated package.xml and setup.py for the new package structure and dependencies.
- Enhanced RViz configuration for improved visualization of the robot and environment.
- Adjusted camera joint parameters in the techtory_franka URDF for better positioning.

File: assembler/techtory_franka_description/urdf/techtory_franka.urdf.xacro (robot description, xacro)
@@ -40,5 +40,5 @@
     <!-- RealSense Cameras -->
     <joint name="camera1_joint" type="fixed">
-        <origin rpy="0 2.356194490192345 0.7853981633974483" xyz="0.65 0.65 2.0"/>
+        <origin rpy="-2.526119746 0.523599 2.186269234" xyz="0.65 0.65 2.0"/>
         <parent link="cell_link"/>
         <child link="camera1_frame"/>
